Commit message: update collision model

File: franka_description/robots/hand.xacro (robot description, xacro)
@@ -17,37 +17,7 @@
       </visual>
       <collision>
-        <origin xyz="0 0 0.04" rpy="0 ${pi/2} ${pi/2}"/>
+        <origin xyz="0 0 0.025" rpy="0 0 0"/>
         <geometry>
-          <cylinder radius="${0.04+safety_distance}" length="0.1" />
-        </geometry>
-      </collision>
-      <collision>
-        <origin xyz="0 -0.05 0.04" rpy="0 0 0"/>
-        <geometry>
-          <sphere radius="${0.04+safety_distance}"  />
-        </geometry>
-      </collision>
-      <collision>
-        <origin xyz="0 0.05 0.04" rpy="0 0 0"/>
-        <geometry>
-          <sphere radius="${0.04+safety_distance}"  />
-        </geometry>
-      </collision>
-      <collision>
-        <origin xyz="0 0 0.1" rpy="0 ${pi/2} ${pi/2}"/>
-        <geometry>
-          <cylinder radius="${0.02+safety_distance}" length="0.1" />
-        </geometry>
-      </collision>
-      <collision>
-        <origin xyz="0 -0.05 0.1" rpy="0 0 0"/>
-        <geometry>
-          <sphere radius="${0.02+safety_distance}"  />
-        </geometry>
-      </collision>
-      <collision>
-        <origin xyz="0 0.05 0.1" rpy="0 0 0"/>
-        <geometry>
-          <sphere radius="${0.02+safety_distance}"  />
+          <box size="${0.045+safety_distance} ${0.21+safety_distance} ${0.09+safety_distance}"  />
         </geometry>
       </collision>
@@ -59,4 +29,10 @@
         </geometry>
       </visual>
+      <collision>
+        <origin xyz="0 0.014 0.03" rpy="0 0 0"/>
+        <geometry>
+          <box size="${0.025+safety_distance} ${0.03+safety_distance} ${0.05+safety_distance}"  />
+        </geometry>
+      </collision>
     </link>
     <link name="${ns}_rightfinger">
@@ -67,4 +43,10 @@
         </geometry>
       </visual>
+      <collision>
+        <origin xyz="0 -0.014 0.03" rpy="0 0 0"/>
+        <geometry>
+          <box size="${0.025+safety_distance} ${0.03+safety_distance} ${0.05+safety_distance}"  />
+        </geometry>
+      </collision>
    </link>
     <joint name="${ns}_finger_joint1" type="prismatic">

File: franka_description/robots/panda_arm.xacro (robot description, xacro)
@@ -1,7 +1,7 @@
 <?xml version='1.0' encoding='utf-8'?>
 <robot xmlns:xacro="http://www.ros.org/wiki/xacro" name="panda">
-  <!-- safety_distance: Minimum safety distance in [m] by which the collision volumes are expanded and which is enforced during robot motions -->
+  <!-- sd: Minimum safety distance in [m] by which the collision volumes are expanded and which is enforced during robot motions -->
   <!-- arm_id: Namespace of the panda arm. Serves to differentiate between arms in case of multiple instances. -->
-  <xacro:macro name="panda_arm" params="arm_id:='panda' description_pkg:='franka_description' connected_to:='' xyz:='0 0 0' rpy:='0 0 0' safety_distance:=0">
+  <xacro:macro name="panda_arm" params="arm_id:='panda' description_pkg:='franka_description' connected_to:='' xyz:='0 0 0' rpy:='0 0 0' sd0:=0 sd1:=0 sd2:=0 sd3:=0 sd4:=0 sd5:=0 sd6:=0 sd7:=0 sd8:=0 cable:=0">
     <xacro:unless value="${not connected_to}">
       <joint name="${arm_id}_joint_${connected_to}" type="fixed">
@@ -18,19 +18,43 @@
       </visual>
       <collision>
+	<!---->
         <origin xyz="-0.075 0 0.06" rpy="0 ${pi/2} 0"/>
         <geometry>
-          <cylinder radius="${0.06+safety_distance}" length="0.03" />
-        </geometry>
-      </collision>
-      <collision>
+          <cylinder radius="${0.06+sd0}" length="0.03" />
+        </geometry>
+      </collision>
+      <collision>
+	<!--base-->
+        <origin xyz="-0.06 0 0.05" rpy="0 0 0"/>
+        <geometry>
+          <box size="${0.24+sd0} ${0.18+sd0} ${0.1+sd0}" />
+        </geometry>
+      </collision>
+      <collision>
+	<!--base+front-->
+        <origin xyz="0.02 0 0.03" rpy="0 0 0"/>
+        <geometry>
+          <cylinder radius="${0.06+sd0}" length="0.06" />
+        </geometry>
+      </collision>
+      <collision>
+	<!--base+cable-->
+        <origin xyz="-0.09 ${-0.075-cable} 0.05" rpy="0 0 0"/>
+        <geometry>
+          <box size="${0.18+sd0} ${0.15+cable+sd0} ${0.1+sd0}" />
+        </geometry>
+      </collision>
+      <collision>
+	<!---->
         <origin xyz="-0.06 0 0.06" rpy="0 0 0"/>
         <geometry>
-          <sphere radius="${0.06+safety_distance}" />
-        </geometry>
-      </collision>
-      <collision>
+          <sphere radius="${0.06+sd0}" />
+        </geometry>
+      </collision>
+      <collision>
+	<!---->
         <origin xyz="-0.09 0 0.06" rpy="0 0 0"/>
         <geometry>
-          <sphere radius="${0.06+safety_distance}" />
+          <sphere radius="${0.06+sd0}" />
         </geometry>
       </collision>
@@ -43,19 +67,29 @@
       </visual>
       <collision>
+	<!---->
         <origin xyz="0 0 -0.1915" rpy="0 0 0"/>
         <geometry>
-          <cylinder radius="${0.06+safety_distance}" length="0.2830" />
-        </geometry>
-      </collision>
-      <collision>
+          <cylinder radius="${0.06+sd1}" length="0.2830" />
+        </geometry>
+      </collision>
+      <collision>
+	<!---->
         <origin xyz="0 0 -0.333" rpy="0 0 0"/>
         <geometry>
-          <sphere radius="${0.06+safety_distance}" />
-        </geometry>
-      </collision>
-      <collision>
+          <sphere radius="${0.06+sd1}" />
+        </geometry>
+      </collision>
+      <collision>
+	<!---->
         <origin xyz="0 0 -0.05" rpy="0 0 0"/>
         <geometry>
-          <sphere radius="${0.06+safety_distance}" />
+          <sphere radius="${0.06+sd1}" />
+        </geometry>
+      </collision>
+      <collision>
+	<!---->
+        <origin xyz="0 -0.05 -0.05" rpy="${pi*30/180} 0 0"/>
+        <geometry>
+          <cylinder radius="${0.055+sd1}" length="0.12" />
         </geometry>
       </collision>
@@ -76,19 +110,29 @@
       </visual>
       <collision>
+	<!---->
+        <origin xyz="0 -0.05 0.05" rpy="${pi*125/180} 0 0"/>
+        <geometry>
+          <cylinder radius="${0.055+sd2}" length="0.12" />
+        </geometry>
+      </collision>
+      <collision>
+	<!---->
         <origin xyz="0 0 0" rpy="0 0 0"/>
         <geometry>
-          <cylinder radius="${0.06+safety_distance}" length="0.12" />
-        </geometry>
-      </collision>
-      <collision>
-        <origin xyz="0 0 -0.06" rpy="0 0 0"/>
-        <geometry>
-          <sphere radius="${0.06+safety_distance}" />
-        </geometry>
-      </collision>
-      <collision>
-        <origin xyz="0 0 0.06" rpy="0 0 0"/>
-        <geometry>
-          <sphere radius="${0.06+safety_distance}" />
+          <cylinder radius="${0.06+sd2}" length="0.12" />
+        </geometry>
+      </collision>
+      <collision>
+	<!---->
+        <origin xyz="0 0 -0.08" rpy="0 0 0"/>
+        <geometry>
+          <sphere radius="${0.06+sd2}" />
+        </geometry>
+      </collision>
+      <collision>
+	<!---->
+        <origin xyz="0 0 0.08" rpy="0 0 0"/>
+        <geometry>
+          <sphere radius="${0.06+sd2}" />
         </geometry>
       </collision>
@@ -109,19 +153,22 @@
       </visual>
       <collision>
+	<!--link3 body-->
         <origin xyz="0 0 -0.145" rpy="0 0 0"/>
         <geometry>
-          <cylinder radius="${0.06+safety_distance}" length="0.15" />
-        </geometry>
-      </collision>
-      <collision>
+          <cylinder radius="${0.06+sd3}" length="0.15" />
+        </geometry>
+      </collision>
+      <collision>
+	<!---->
         <origin xyz="0 0 -0.22" rpy="0 0 0"/>
         <geometry>
-          <sphere radius="${0.06+safety_distance}" />
-        </geometry>
-      </collision>
-      <collision>
+          <sphere radius="${0.06+sd3}" />
+        </geometry>
+      </collision>
+      <collision>
+	<!---->
         <origin xyz="0 0 -0.07" rpy="0 0 0"/>
         <geometry>
-          <sphere radius="${0.06+safety_distance}" />
+          <sphere radius="${0.06+sd3}" />
         </geometry>
       </collision>
@@ -142,19 +189,36 @@
       </visual>
       <collision>
+	<!--link4 body-->
         <origin xyz="0 0 0" rpy="0 0 0"/>
         <geometry>
-          <cylinder radius="${0.06+safety_distance}" length="0.12" />
-        </geometry>
-      </collision>
-      <collision>
+          <cylinder radius="${0.06+sd4}" length="0.12" />
+        </geometry>
+      </collision>
+      <collision>
+	<!---->
         <origin xyz="0 0 0.06" rpy="0 0 0"/>
         <geometry>
-          <sphere radius="${0.06+safety_distance}" />
-        </geometry>
-      </collision>
-      <collision>
+          <sphere radius="${0.06+sd4}" />
+        </geometry>
+      </collision>
+      <collision>
+	<!---->
+        <origin xyz="-0.01 0.01 0.07" rpy="0 0 0"/>
+        <geometry>
+          <cylinder radius="${0.06+sd4}" length="0.02" />
+        </geometry>
+      </collision>
+      <collision>
+	<!---->
+        <origin xyz="0.01 -0.01 -0.07" rpy="0 0 0"/>
+        <geometry>
+          <cylinder radius="${0.06+sd4}" length="0.02" />
+        </geometry>
+      </collision>
+      <collision>
+	<!---->
         <origin xyz="0 0 -0.06" rpy="0 0 0"/>
         <geometry>
-          <sphere radius="${0.06+safety_distance}" />
+          <sphere radius="${0.06+sd4}" />
         </geometry>
       </collision>
@@ -175,37 +239,43 @@
       </visual>
       <collision>
+	<!---->
         <origin xyz="0 0 -0.26" rpy="0 0 0"/>
         <geometry>
-          <cylinder radius="${0.06+safety_distance}" length="0.1" />
-        </geometry>
-      </collision>
-      <collision>
-        <origin xyz="0 0 -0.31" rpy="0 0 0"/>
-        <geometry>
-          <sphere radius="${0.06+safety_distance}" />
-        </geometry>
-      </collision>
-      <collision>
-        <origin xyz="0 0 -0.21" rpy="0 0 0"/>
-        <geometry>
-          <sphere radius="${0.06+safety_distance}" />
-        </geometry>
-      </collision>
-      <collision>
-        <origin xyz="0 0.08 -0.13" rpy="0 0 0"/>
-        <geometry>
-          <cylinder radius="${0.025+safety_distance}" length="0.14" />
-        </geometry>
-      </collision>
-      <collision>
-        <origin xyz="0 0.08 -0.06" rpy="0 0 0"/>
-        <geometry>
-          <sphere radius="${0.025+safety_distance}" />
-        </geometry>
-      </collision>
-      <collision>
-        <origin xyz="0 0.08 -0.20" rpy="0 0 0"/>
-        <geometry>
-          <sphere radius="${0.025+safety_distance}" />
+          <cylinder radius="${0.06+sd5}" length="0.1" />
+        </geometry>
+      </collision>
+      <collision>
+	<!--almost link 4-->
+        <origin xyz="0 0 -0.32" rpy="0 0 0"/>
+        <geometry>
+          <sphere radius="${0.06+sd5}" />
+        </geometry>
+      </collision>
+      <collision>
+	<!---->
+        <origin xyz="0 0 -0.22" rpy="0 0 0"/>
+        <geometry>
+          <sphere radius="${0.06+sd5}" />
+        </geometry>
+      </collision>
+      <collision>
+	<!--link5 long body part-->
+        <origin xyz="0 0.08 -0.12" rpy="${-pi*8/180} 0 0"/>
+        <geometry>
+          <cylinder radius="${0.035+sd5}" length="0.17" />
+        </geometry>
+      </collision>
+      <collision>
+	<!--curve part-->
+        <origin xyz="0 0.085 0" rpy="0 0 0"/>
+        <geometry>
+          <sphere radius="${0.06+sd5}" />
+        </geometry>
+      </collision>
+      <collision>
+	<!---->
+        <origin xyz="0 0.05 -0.19" rpy="0 0 0"/>
+        <geometry>
+          <sphere radius="${0.05+sd5}" />
         </geometry>
       </collision>
@@ -226,19 +296,29 @@
       </visual>
       <collision>
+	<!---->
         <origin xyz="0 0 -0.03" rpy="0 0 0"/>
         <geometry>
-          <cylinder radius="${0.05+safety_distance}" length="0.08" />
-        </geometry>
-      </collision>
-      <collision>
+          <cylinder radius="${0.06+sd6}" length="0.08" />
+        </geometry>
+      </collision>
+      <collision>
+	<!---->
+        <origin xyz="0.02 0 0.01" rpy="0 ${pi/2} 0"/>
+        <geometry>
+          <cylinder radius="${0.06+sd6}" length="0.07" />
+        </geometry>
+      </collision>
+      <collision>
+	<!--curve part-->
         <origin xyz="0 0 0.01" rpy="0 0 0"/>
         <geometry>
-          <sphere radius="${0.05+safety_distance}" />
-        </geometry>
-      </collision>
-      <collision>
-        <origin xyz="0 0 -0.07" rpy="0 0 0"/>
-        <geometry>
-          <sphere radius="${0.05+safety_distance}" />
+          <sphere radius="${0.06+sd6}" />
+        </geometry>
+      </collision>
+      <collision>
+	<!--link6and5 connection part-->
+        <origin xyz="0 0 -0.08" rpy="0 0 0"/>
+        <geometry>
+          <sphere radius="${0.051+sd6}" />
         </geometry>
       </collision>
@@ -259,19 +339,22 @@
       </visual>
       <collision>
+	<!--link7's body-->
         <origin xyz="0 0 0.01" rpy="0 0 0"/>
         <geometry>
-          <cylinder radius="${0.04+safety_distance}" length="0.14" />
-        </geometry>
-      </collision>
-      <collision>
+          <cylinder radius="${0.045+sd7}" length="0.14" />
+        </geometry>
+      </collision>
+      <collision>
+	<!--link7and8 connection part-->
         <origin xyz="0 0 0.08" rpy="0 0 0"/>
         <geometry>
-          <sphere radius="${0.04+safety_distance}"  />
-        </geometry>
-      </collision>
-      <collision>
+          <sphere radius="${0.04+sd7}"  />
+        </geometry>
+      </collision>
+      <collision>
+	<!--button part-->
         <origin xyz="0 0 -0.06" rpy="0 0 0"/>
         <geometry>
-          <sphere radius="${0.04+safety_distance}"  />
+          <sphere radius="${0.045+sd7}"  />
         </geometry>
       </collision>
@@ -287,19 +370,15 @@
     <link name="${arm_id}_link8">
       <collision>
-        <origin xyz="0.0424 0.0424 -0.0250" rpy="${pi} ${pi/2} ${pi/2}"/>
-        <geometry>
-          <cylinder radius="${0.03+safety_distance}"  length="0.01" />
-        </geometry>
-      </collision>
-      <collision>
-        <origin xyz="0.0424 0.0424 -0.02" rpy="0 0 0"/>
-        <geometry>
-          <sphere radius="${0.03+safety_distance}"  />
-        </geometry>
-      </collision>
-      <collision>
-        <origin xyz="0.0424 0.0424 -0.03" rpy="0 0 0"/>
-        <geometry>
-          <sphere radius="${0.03+safety_distance}"  />
+	<!--button part-->
+        <origin xyz="0.04 0.04 -0.03" rpy="0 0 ${pi/4}"/>
+        <geometry>
+          <box size="${0.07+sd8} ${0.07+sd8} ${0.02+sd8}" />
+        </geometry>
+      </collision>
+      <collision>
+	<!--rotate part-->
+        <origin xyz="0 0 -0.028" rpy="0 0 0"/>
+        <geometry>
+          <cylinder radius="${0.05+sd8}"  length="0.05"  />
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