Commit message: update custom changes

File: franka_description/robots/panda_arm.xacro (robot description, xacro)
@@ -1,5 +1,7 @@
 <?xml version='1.0' encoding='utf-8'?>
 <robot xmlns:xacro="http://www.ros.org/wiki/xacro" name="panda">
-  <xacro:macro name="panda_arm" params="arm_id:='panda' description_pkg:='franka_description' connected_to:='' xyz:='0 0 0' rpy:='0 0 0'">
+  <!-- safety_distance: Minimum safety distance in [m] by which the collision volumes are expanded and which is enforced during robot motions -->
+  <!-- arm_id: Namespace of the panda arm. Serves to differentiate between arms in case of multiple instances. -->
+  <xacro:macro name="panda_arm" params="arm_id:='panda' description_pkg:='franka_description' connected_to:='' xyz:='0 0 0' rpy:='0 0 0' safety_distance:=0.02">
     <xacro:unless value="${not connected_to}">
       <joint name="${arm_id}_joint_${connected_to}" type="fixed">
@@ -16,6 +18,19 @@
       </visual>
       <collision>
-        <geometry>
-          <mesh filename="package://${description_pkg}/meshes/collision/link0.stl"/>
+        <origin xyz="-0.075 0 0.06" rpy="0 ${pi/2} 0"/>
+        <geometry>
+          <cylinder radius="${0.06+safety_distance}" length="0.03" />
+        </geometry>
+      </collision>
+      <collision>
+        <origin xyz="-0.06 0 0.06" rpy="0 0 0"/>
+        <geometry>
+          <sphere radius="${0.06+safety_distance}" />
+        </geometry>
+      </collision>
+      <collision>
+        <origin xyz="-0.09 0 0.06" rpy="0 0 0"/>
+        <geometry>
+          <sphere radius="${0.06+safety_distance}" />
         </geometry>
       </collision>
@@ -28,6 +43,19 @@
       </visual>
       <collision>
-        <geometry>
-          <mesh filename="package://${description_pkg}/meshes/collision/link1.stl"/>
+        <origin xyz="0 0 -0.1915" rpy="0 0 0"/>
+        <geometry>
+          <cylinder radius="${0.06+safety_distance}" length="0.2830" />
+        </geometry>
+      </collision>
+      <collision>
+        <origin xyz="0 0 -0.333" rpy="0 0 0"/>
+        <geometry>
+          <sphere radius="${0.06+safety_distance}" />
+        </geometry>
+      </collision>
+      <collision>
+        <origin xyz="0 0 -0.05" rpy="0 0 0"/>
+        <geometry>
+          <sphere radius="${0.06+safety_distance}" />
         </geometry>
       </collision>
@@ -48,6 +76,19 @@
       </visual>
       <collision>
-        <geometry>
-          <mesh filename="package://${description_pkg}/meshes/collision/link2.stl"/>
+        <origin xyz="0 0 0" rpy="0 0 0"/>
+        <geometry>
+          <cylinder radius="${0.06+safety_distance}" length="0.12" />
+        </geometry>
+      </collision>
+      <collision>
+        <origin xyz="0 0 -0.06" rpy="0 0 0"/>
+        <geometry>
+          <sphere radius="${0.06+safety_distance}" />
+        </geometry>
+      </collision>
+      <collision>
+        <origin xyz="0 0 0.06" rpy="0 0 0"/>
+        <geometry>
+          <sphere radius="${0.06+safety_distance}" />
         </geometry>
       </collision>
@@ -68,6 +109,19 @@
       </visual>
       <collision>
-        <geometry>
-          <mesh filename="package://${description_pkg}/meshes/collision/link3.stl"/>
+        <origin xyz="0 0 -0.145" rpy="0 0 0"/>
+        <geometry>
+          <cylinder radius="${0.06+safety_distance}" length="0.15" />
+        </geometry>
+      </collision>
+      <collision>
+        <origin xyz="0 0 -0.22" rpy="0 0 0"/>
+        <geometry>
+          <sphere radius="${0.06+safety_distance}" />
+        </geometry>
+      </collision>
+      <collision>
+        <origin xyz="0 0 -0.07" rpy="0 0 0"/>
+        <geometry>
+          <sphere radius="${0.06+safety_distance}" />
         </geometry>
       </collision>
@@ -88,6 +142,19 @@
       </visual>
       <collision>
-        <geometry>
-          <mesh filename="package://${description_pkg}/meshes/collision/link4.stl"/>
+        <origin xyz="0 0 0" rpy="0 0 0"/>
+        <geometry>
+          <cylinder radius="${0.06+safety_distance}" length="0.12" />
+        </geometry>
+      </collision>
+      <collision>
+        <origin xyz="0 0 0.06" rpy="0 0 0"/>
+        <geometry>
+          <sphere radius="${0.06+safety_distance}" />
+        </geometry>
+      </collision>
+      <collision>
+        <origin xyz="0 0 -0.06" rpy="0 0 0"/>
+        <geometry>
+          <sphere radius="${0.06+safety_distance}" />
         </geometry>
       </collision>
@@ -108,6 +175,37 @@
       </visual>
       <collision>
-        <geometry>
-          <mesh filename="package://${description_pkg}/meshes/collision/link5.stl"/>
+        <origin xyz="0 0 -0.26" rpy="0 0 0"/>
+        <geometry>
+          <cylinder radius="${0.06+safety_distance}" length="0.1" />
+        </geometry>
+      </collision>
+      <collision>
+        <origin xyz="0 0 -0.31" rpy="0 0 0"/>
+        <geometry>
+          <sphere radius="${0.06+safety_distance}" />
+        </geometry>
+      </collision>
+      <collision>
+        <origin xyz="0 0 -0.21" rpy="0 0 0"/>
+        <geometry>
+          <sphere radius="${0.06+safety_distance}" />
+        </geometry>
+      </collision>
+      <collision>
+        <origin xyz="0 0.08 -0.13" rpy="0 0 0"/>
+        <geometry>
+          <cylinder radius="${0.025+safety_distance}" length="0.14" />
+        </geometry>
+      </collision>
+      <collision>
+        <origin xyz="0 0.08 -0.06" rpy="0 0 0"/>
+        <geometry>
+          <sphere radius="${0.025+safety_distance}" />
+        </geometry>
+      </collision>
+      <collision>
+        <origin xyz="0 0.08 -0.20" rpy="0 0 0"/>
+        <geometry>
+          <sphere radius="${0.025+safety_distance}" />
         </geometry>
       </collision>
@@ -128,6 +226,19 @@
       </visual>
       <collision>
-        <geometry>
-          <mesh filename="package://${description_pkg}/meshes/collision/link6.stl"/>
+        <origin xyz="0 0 -0.03" rpy="0 0 0"/>
+        <geometry>
+          <cylinder radius="${0.05+safety_distance}" length="0.08" />
+        </geometry>
+      </collision>
+      <collision>
+        <origin xyz="0 0 0.01" rpy="0 0 0"/>
+        <geometry>
+          <sphere radius="${0.05+safety_distance}" />
+        </geometry>
+      </collision>
+      <collision>
+        <origin xyz="0 0 -0.07" rpy="0 0 0"/>
+        <geometry>
+          <sphere radius="${0.05+safety_distance}" />
         </geometry>
       </collision>
@@ -148,6 +259,19 @@
       </visual>
       <collision>
-        <geometry>
-          <mesh filename="package://${description_pkg}/meshes/collision/link7.stl"/>
+        <origin xyz="0 0 0.01" rpy="0 0 0"/>
+        <geometry>
+          <cylinder radius="${0.04+safety_distance}" length="0.14" />
+        </geometry>
+      </collision>
+      <collision>
+        <origin xyz="0 0 0.08" rpy="0 0 0"/>
+        <geometry>
+          <sphere radius="${0.04+safety_distance}"  />
+        </geometry>
+      </collision>
+      <collision>
+        <origin xyz="0 0 -0.06" rpy="0 0 0"/>
+        <geometry>
+          <sphere radius="${0.04+safety_distance}"  />
         </geometry>
       </collision>
@@ -161,10 +285,28 @@
       <limit effort="12" lower="-2.8973" upper="2.8973" velocity="2.6100"/>
     </joint>
-    <link name="${arm_id}_link8"/>
+    <link name="${arm_id}_link8">
+      <collision>
+        <origin xyz="0.0424 0.0424 -0.0250" rpy="${pi} ${pi/2} ${pi/2}"/>
+        <geometry>
+          <cylinder radius="${0.03+safety_distance}"  length="0.01" />
+        </geometry>
+      </collision>
+      <collision>
+        <origin xyz="0.0424 0.0424 -0.02" rpy="0 0 0"/>
+        <geometry>
+          <sphere radius="${0.03+safety_distance}"  />
+        </geometry>
+      </collision>
+      <collision>
+        <origin xyz="0.0424 0.0424 -0.03" rpy="0 0 0"/>
+        <geometry>
+          <sphere radius="${0.03+safety_distance}"  />
+        </geometry>
+      </collision>
+    </link>
     <joint name="${arm_id}_joint8" type="fixed">
       <origin rpy="0 0 0" xyz="0 0 0.107"/>
       <parent link="${arm_id}_link7"/>
       <child link="${arm_id}_link8"/>
-      <axis xyz="0 0 0"/>
     </joint>
   </xacro:macro>

Commit message: update custom mesh properties

File: franka_description/robots/panda_arm.xacro (robot description, xacro)
@@ -276,4 +276,9 @@
         </geometry>
       </collision>
+      <collision>
+        <geometry>
+          <mesh filename="package://${description_pkg}/meshes/collision/link7.stl"/>
+        </geometry>
+      </collision>
     </link>
     <joint name="${arm_id}_joint7" type="revolute">
@@ -286,22 +291,4 @@
     </joint>
     <link name="${arm_id}_link8">
-      <collision>
-        <origin xyz="0.0424 0.0424 -0.0250" rpy="${pi} ${pi/2} ${pi/2}"/>
-        <geometry>
-          <cylinder radius="${0.03+safety_distance}"  length="0.01" />
-        </geometry>
-      </collision>
-      <collision>
-        <origin xyz="0.0424 0.0424 -0.02" rpy="0 0 0"/>
-        <geometry>
-          <sphere radius="${0.03+safety_distance}"  />
-        </geometry>
-      </collision>
-      <collision>
-        <origin xyz="0.0424 0.0424 -0.03" rpy="0 0 0"/>
-        <geometry>
-          <sphere radius="${0.03+safety_distance}"  />
-        </geometry>
-      </collision>
     </link>
     <joint name="${arm_id}_joint8" type="fixed">

Commit message: update joint limit

File: franka_description/robots/panda_arm.xacro (robot description, xacro)
@@ -100,5 +100,6 @@
       <child link="${arm_id}_link2"/>
       <axis xyz="0 0 1"/>
-      <limit effort="87" lower="-1.7628" upper="1.7628" velocity="2.1750"/>
+      <limit effort="87" lower="-1.4628" upper="1.4628" velocity="2.1750"/>
+      <!-- <limit effort="87" lower="-1.7628" upper="1.7628" velocity="2.1750"/> -->
     </joint>
     <link name="${arm_id}_link3">

Commit message: joint limit (prevent self collision)

File: franka_description/robots/panda_arm.xacro (robot description, xacro)
@@ -330,5 +330,6 @@
       <child link="${arm_id}_link6"/>
       <axis xyz="0 0 1"/>
-      <limit effort="12" lower="-0.0175" upper="3.7525" velocity="2.6100"/>
+      <!-- <limit effort="12" lower="-0.0175" upper="3.7525" velocity="2.6100"/> -->
+      <limit effort="12" lower="0.75" upper="3.7525" velocity="2.6100"/>
     </joint>
     <link name="${arm_id}_link7">

Commit message: update params

File: franka_description/robots/panda_arm.xacro (robot description, xacro)
@@ -330,6 +330,6 @@
       <child link="${arm_id}_link6"/>
       <axis xyz="0 0 1"/>
-      <!-- <limit effort="12" lower="-0.0175" upper="3.7525" velocity="2.6100"/> -->
-      <limit effort="12" lower="0.75" upper="3.7525" velocity="2.6100"/>
+      <limit effort="12" lower="-0.0175" upper="3.7525" velocity="2.6100"/>
+      <!-- <limit effort="12" lower="0.75" upper="3.7525" velocity="2.6100"/> -->
     </joint>
     <link name="${arm_id}_link7">

File: franka_description/robots/panda_arm_hand.urdf.xacro (robot description, xacro)
@@ -3,5 +3,5 @@
   <xacro:include filename="$(find franka_description)/robots/panda_arm.xacro"/>
   <xacro:include filename="$(find franka_description)/robots/hand.xacro"/>
-  <xacro:panda_arm safety_distance="0.03"/>
+  <xacro:panda_arm safety_distance="0.03"/>-->
   <xacro:hand ns="panda" rpy="0 0 ${-pi/4}" connected_to="panda_link8" safety_distance="0.03"/>
 </robot>

Commit message: update dh params

File: franka_description/robots/panda_arm.xacro (robot description, xacro)
@@ -3,5 +3,5 @@
   <!-- sd: Minimum safety distance in [m] by which the collision volumes are expanded and which is enforced during robot motions -->
   <!-- arm_id: Namespace of the panda arm. Serves to differentiate between arms in case of multiple instances. -->
-  <xacro:macro name="panda_arm" params="arm_id:='panda' description_pkg:='franka_description' connected_to:='' xyz:='0 0 0' rpy:='0 0 0' sd0:=0 sd1:=0 sd2:=0 sd3:=0 sd4:=0 sd5:=0 sd6:=0 sd7:=0 sd8:=0 cable:=0">
+  <xacro:macro name="panda_arm" params="arm_id:='panda' description_pkg:='franka_description' connected_to:='' xyz:='0 0 0' rpy:='0 0 0' sd0:=0 sd1:=0 sd2:=0 sd3:=0 sd4:=0 sd5:=0 sd6:=0 sd7:=0 sd8:=0 cable:=0 a1:=0 d1:=0 theta1:=0 alpha1:=0 a2:=0 d2:=0 theta2:=0 alpha2:=0 a3:=0 d3:=0 theta3:=0 alpha3:=0 a4:=0 d4:=0 theta4:=0 alpha4:=0 a5:=0 d5:=0 theta5:=0 alpha5:=0 a6:=0 d6:=0 theta6:=0 alpha6:=0 a7:=0 d7:=0 theta7:=0 alpha7:=0 ">
     <xacro:unless value="${not connected_to}">
       <joint name="${arm_id}_joint_${connected_to}" type="fixed">
@@ -95,8 +95,15 @@
       </collision>
     </link>
+    <link name="${arm_id}_link1_augmented">
+    </link>
+    <joint name="${arm_id}_joint1_augmented" type="fixed">
+      <origin xyz="${a1} 0 0" rpy="${alpha1} 0 0"/>
+      <parent link="${arm_id}_link0" />
+      <child link="${arm_id}_link1_augmented" />
+    </joint>
     <joint name="${arm_id}_joint1" type="revolute">
       <safety_controller k_position="100.0" k_velocity="40.0" soft_lower_limit="-2.8973" soft_upper_limit="2.8973"/>
-      <origin rpy="0 0 0" xyz="0 0 0.333"/>
-      <parent link="${arm_id}_link0"/>
+      <origin rpy="0 0 ${theta1}" xyz="0 0 ${0.333+d1}"/>
+      <parent link="${arm_id}_link1_augmented"/>
       <child link="${arm_id}_link1"/>
       <axis xyz="0 0 1"/>
@@ -138,8 +145,15 @@
       </collision>
     </link>
+    <link name="${arm_id}_link2_augmented">
+    </link>
+    <joint name="${arm_id}_joint2_augmented" type="fixed">
+      <origin xyz="${a2} 0 0" rpy="${-pi/2+alpha2} 0 0"/>
+      <parent link="${arm_id}_link1" />
+      <child link="${arm_id}_link2_augmented" />
+    </joint>
     <joint name="${arm_id}_joint2" type="revolute">
       <safety_controller k_position="100.0" k_velocity="40.0" soft_lower_limit="-1.7628" soft_upper_limit="1.7628"/>
-      <origin rpy="${-pi/2} 0 0" xyz="0 0 0"/>
-      <parent link="${arm_id}_link1"/>
+      <origin rpy="0 0 ${theta2}" xyz="0 0 ${d2}"/>
+      <parent link="${arm_id}_link2_augmented"/>
       <child link="${arm_id}_link2"/>
       <axis xyz="0 0 1"/>
@@ -174,8 +188,15 @@
       </collision>
     </link>
+    <link name="${arm_id}_link3_augmented">
+    </link>
+    <joint name="${arm_id}_joint3_augmented" type="fixed">
+      <origin xyz="${a3} 0 0" rpy="${pi/2+alpha3} 0 0"/>
+      <parent link="${arm_id}_link2" />
+      <child link="${arm_id}_link3_augmented" />
+    </joint>
     <joint name="${arm_id}_joint3" type="revolute">
       <safety_controller k_position="100.0" k_velocity="40.0" soft_lower_limit="-2.8973" soft_upper_limit="2.8973"/>
-      <origin rpy="${pi/2} 0 0" xyz="0 -0.316 0"/>
-      <parent link="${arm_id}_link2"/>
+      <origin rpy="0 0 ${theta3}" xyz="0 0 ${0.316+d3}"/>
+      <parent link="${arm_id}_link3_augmented"/>
       <child link="${arm_id}_link3"/>
       <axis xyz="0 0 1"/>
@@ -224,8 +245,15 @@
       </collision>
     </link>
+    <link name="${arm_id}_link4_augmented">
+    </link>
+    <joint name="${arm_id}_joint4_augmented" type="fixed">
+      <origin xyz="${0.0825+a4} 0 0" rpy="${pi/2+alpha4} 0 0"/>
+      <parent link="${arm_id}_link3" />
+      <child link="${arm_id}_link4_augmented" />
+    </joint>
     <joint name="${arm_id}_joint4" type="revolute">
       <safety_controller k_position="100.0" k_velocity="40.0" soft_lower_limit="-3.0718" soft_upper_limit="-0.0698"/>
-      <origin rpy="${pi/2} 0 0" xyz="0.0825 0 0"/>
-      <parent link="${arm_id}_link3"/>
+      <origin rpy="0 0 ${theta4}" xyz="0 0 ${d4}"/>
+      <parent link="${arm_id}_link4_augmented"/>
       <child link="${arm_id}_link4"/>
       <axis xyz="0 0 1"/>
@@ -281,8 +309,15 @@
       </collision>
     </link>
+    <link name="${arm_id}_link5_augmented">
+    </link>
+    <joint name="${arm_id}_joint5_augmented" type="fixed">
+      <origin xyz="${-0.0825+a5} 0 0" rpy="${-pi/2+alpha5} 0 0"/>
+      <parent link="${arm_id}_link4" />
+      <child link="${arm_id}_link5_augmented" />
+    </joint>
     <joint name="${arm_id}_joint5" type="revolute">
       <safety_controller k_position="100.0" k_velocity="40.0" soft_lower_limit="-2.8973" soft_upper_limit="2.8973"/>
-      <origin rpy="${-pi/2} 0 0" xyz="-0.0825 0.384 0"/>
-      <parent link="${arm_id}_link4"/>
+      <origin rpy="0 0 ${theta5}" xyz="0 0 ${0.384+d5}"/>
+      <parent link="${arm_id}_link5_augmented"/>
       <child link="${arm_id}_link5"/>
       <axis xyz="0 0 1"/>
@@ -324,8 +359,15 @@
       </collision>
     </link>
+    <link name="${arm_id}_link6_augmented">
+    </link>
+    <joint name="${arm_id}_joint6_augmented" type="fixed">
+      <origin xyz="${a6} 0 0" rpy="${pi/2+alpha6} 0 0"/>
+      <parent link="${arm_id}_link5" />
+      <child link="${arm_id}_link6_augmented" />
+    </joint>
     <joint name="${arm_id}_joint6" type="revolute">
       <safety_controller k_position="100.0" k_velocity="40.0" soft_lower_limit="-0.0175" soft_upper_limit="3.7525"/>
-      <origin rpy="${pi/2} 0 0" xyz="0 0 0"/>
-      <parent link="${arm_id}_link5"/>
+      <origin rpy="0 0 ${theta6}" xyz="0 0 ${d6}"/>
+      <parent link="${arm_id}_link6_augmented"/>
       <child link="${arm_id}_link6"/>
       <axis xyz="0 0 1"/>
@@ -361,8 +403,15 @@
       </collision>
     </link>
+    <link name="${arm_id}_link7_augmented">
+    </link>
+    <joint name="${arm_id}_joint7_augmented" type="fixed">
+      <origin xyz="${0.088+a7} 0 0" rpy="${pi/2+alpha7} 0 0"/>
+      <parent link="${arm_id}_link6" />
+      <child link="${arm_id}_link7_augmented" />
+    </joint>
     <joint name="${arm_id}_joint7" type="revolute">
       <safety_controller k_position="100.0" k_velocity="40.0" soft_lower_limit="-2.8973" soft_upper_limit="2.8973"/>
-      <origin rpy="${pi/2} 0 0" xyz="0.088 0 0"/>
-      <parent link="${arm_id}_link6"/>
+      <origin rpy="0 0 ${theta7}" xyz="0 0 ${d7}"/>
+      <parent link="${arm_id}_link7_augmented"/>
       <child link="${arm_id}_link7"/>
       <axis xyz="0 0 1"/>
